Commit message: 添加chassis_control

File: xacro/sentry.xacro (robot description, xacro)
@@ -1,12 +1,13 @@
 <?xml version="1.0" encoding="utf-8"?>
 <robot name="sentry" xmlns:xacro="http://www.ros.org/wiki/xacro">
-    <xacro:include filename="$(find sentry9)/xacro/sentry_chassis.xacro" />
+    <xacro:include filename="$(find sentry9)/xacro/sentry_chassis_new.xacro" />
     <xacro:include filename="$(find sentry9)/xacro/sentry_yaw.xacro" />
+    <!--xacro:include filename="$(find sentry9)/xacro/sentry_laser.xacro" /-->
     <xacro:include filename="$(find sentry9)/xacro/sentry_pitch.xacro" />
-    <!--xacro:include filename="$(find sentry9)/xacro/sentry_laser.xacro" /-->
     <xacro:include filename="$(find sentry9)/xacro/sentry_camera.xacro" />
     <xacro:include filename="$(find sentry9)/xacro/sentry_imu.xacro" />
     <xacro:include filename="$(find sentry9)/xacro/sentry_trigger.xacro" />
     <xacro:include filename="$(find sentry9)/xacro/livox_sim.xacro"/>
+    <xacro:include filename="$(find sentry9)/xacro/sentry_wheel.xacro" />
     <!-- Yaw_Joint -->
   <joint
@@ -60,4 +61,9 @@
     <axis xyz="0 0 -1" />
   </joint>
+<xacro:sentry_wheel heading_name="Heading_Left_Front" driving_name="Driving_Left_Front" x='0.178' y= '0.178' z='0.042' />
+<xacro:sentry_wheel heading_name="Heading_Left_Back" driving_name="Driving_Left_Back" x='-0.178' y= '0.178' z='0.042' />
+<xacro:sentry_wheel heading_name="Heading_Right_Front" driving_name="Driving_Right_Front" x='0.178' y= '-0.178' z='0.042' />
+<xacro:sentry_wheel heading_name="Heading_Right_Back" driving_name="Driving_Right_Back" x='-0.178' y= '-0.178' z='0.042' />
+<!-- transmission for left_back_wheel-->
     <!-- controller -->
   <gazebo>

File: xacro/sentry_wheel.xacro (robot description, xacro)
@@ -1,59 +1,18 @@
-<?xml version="1.0" encoding="utf-8"?>
-<robot name="sentry_chassis"   xmlns:xacro="http://www.ros.org/wiki/xacro">
-<link
-    name="base_link">
-    <inertial>
-      <origin
-        xyz="0.00225297070027259 0.0021561284245786 0.0235031309630918"
-        rpy="0 0 0" />
-      <mass
-        value="4.42503101633294" />
-      <inertia
-        ixx="0.0160955362042838"
-        ixy="-4.37751798666585E-07"
-        ixz="-3.76131129209663E-05"
-        iyy="0.00951260621260376"
-        iyz="-1.23241554900005E-05"
-        izz="0.0235407659569457" />
-    </inertial>
-    <visual>
-      <origin
-        xyz="0 0 0"
-        rpy="0 0 0" />
-      <geometry>
-        <mesh
-          filename="package://sentry9/meshes/base_link.STL" />
-      </geometry>
-      <material
-        name="">
-        <color
-          rgba="1 1 1 1" />
-      </material>
-    </visual>
-    <collision>
-      <origin
-        xyz="0 0 0"
-        rpy="0 0 0" />
-      <geometry>
-        <mesh
-          filename="package://sentry9/meshes/base_link.STL" />
-      </geometry>
-    </collision>
-  </link>
-<link name="base_footprint">
-   </link>
-  <joint
-    name="footprint2baselink"
-    type="fixed">
-    <origin
-      xyz="0 0 0.3"
-      rpy="0 0 0" />
-    <parent
-      link="base_footprint" />
-    <child
-      link="base_link" />
-  </joint>
-  <link
-    name="Heading_Left_Front_Link">
+<?xml version="1.0"?>
+<robot xmlns:xacro="http://ros.org/wiki/xacro">
+  <xacro:macro name="joint_transmission" params="prefix">
+    <transmission name="trans_${prefix}">
+      <type>transmission_interface/SimpleTransmission</type>
+      <actuator name="${prefix}_actuator">
+        <mechanicalReduction>1</mechanicalReduction>
+      </actuator>
+      <joint name="${prefix}_Joint">
+        <hardwareInterface>hardware_interface/EffortJointInterface</hardwareInterface>
+      </joint>
+    </transmission>
+  </xacro:macro>
+  <xacro:macro name="sentry_wheel" params="heading_name driving_name x y z">
+    <link
+    name="${heading_name}_Link">
     <inertial>
       <origin
@@ -95,18 +54,18 @@
   </link>
   <joint
-    name="Heading_Left_Front_Joint"
+    name="${heading_name}_Joint"
     type="continuous">
     <origin
-      xyz="0.178 0.178 0.042"
+      xyz="${x}  ${y} ${z}"
       rpy="0 0 0" />
     <parent
       link="base_link" />
     <child
-      link="Heading_Left_Front_Link" />
+      link="${heading_name}_Link" />
     <axis
       xyz="0 0 1" />
   </joint>
   <link
-    name="Driving_Left_Front_Link">
+    name="${driving_name}_Link">
     <inertial>
       <origin
@@ -148,5 +107,5 @@
   </link>
   <joint
-    name="Driving_Left_Front_Joint"
+    name="${driving_name}_Joint"
     type="revolute">
     <origin
@@ -154,10 +113,13 @@
       rpy="0 0 0" />
     <parent
-      link="Heading_Left_Front_Link" />
+      link="${heading_name}_Link" />
     <child
-      link="Driving_Left_Front_Link" />
+      link="${driving_name}_Link" />
     <axis
       xyz="-0.14817 -0.98896 0" />
     <limit lower="-1e9" upper="1e9" effort="10" velocity="70" />
   </joint>
+  <xacro:joint_transmission prefix="${heading_name}"/>
+  <xacro:joint_transmission prefix="${driving_name}"/>
+  </xacro:macro>
 </robot>

Commit message: 10.30

File: xacro/sentry.xacro (robot description, xacro)
@@ -65,5 +65,40 @@
 <xacro:sentry_wheel heading_name="Heading_Right_Front" driving_name="Driving_Right_Front" x='0.178' y= '-0.178' z='0.042' />
 <xacro:sentry_wheel heading_name="Heading_Right_Back" driving_name="Driving_Right_Back" x='-0.178' y= '-0.178' z='0.042' />
-<!-- transmission for left_back_wheel-->
+ <gazebo reference="base_link">
+     <material>Gazebo/Grey</material>
+     <turnGravityOff>false</turnGravityOff>
+ </gazebo>
+   <gazebo reference="Heading_Left_Front_Link">
+     <material>Gazebo/White</material>
+     <turnGravityOff>false</turnGravityOff>
+ </gazebo>
+   <gazebo reference="Heading_Left_Back_Link">
+     <material>Gazebo/White</material>
+     <turnGravityOff>false</turnGravityOff>
+ </gazebo>
+   <gazebo reference="Heading_Right_Front_Link">
+     <material>Gazebo/White</material>
+     <turnGravityOff>false</turnGravityOff>
+ </gazebo>
+   <gazebo reference="Heading_Right_Back_Link">
+     <material>Gazebo/White</material>
+     <turnGravityOff>false</turnGravityOff>
+ </gazebo>
+   <gazebo reference="Driving_Left_Front_Link">
+     <material>Gazebo/Grey</material>
+     <turnGravityOff>false</turnGravityOff>
+ </gazebo>
+   <gazebo reference="Driving_Left_back_Link">
+     <material>Gazebo/Grey</material>
+     <turnGravityOff>false</turnGravityOff>
+ </gazebo>
+    <gazebo reference="Driving_Right_Front_Link">
+     <material>Gazebo/Grey</material>
+     <turnGravityOff>false</turnGravityOff>
+ </gazebo>
+   <gazebo reference="Driving_Right_Back_Link">
+     <material>Gazebo/Grey</material>
+     <turnGravityOff>false</turnGravityOff>
+ </gazebo>
     <!-- controller -->
   <gazebo>
