Commit message: gmapping建图,保存地图

File: src/sentry_laser_sim/xacro/laser.xacro (robot description, xacro)
@@ -8,5 +8,5 @@
   <xacro:property name="laser_min_range" value="0.1"/>
   <xacro:property name="laser_max_range" value="200.0"/>
-  <xacro:property name="ros_topic" value="scan"/>
+  <xacro:property name="ros_topic" value="scan1"/>
   <xacro:property name="samples" value="10000"/>
   <xacro:property name="downsample" value="0"/>
@@ -35,5 +35,5 @@
 				</horizontal>
 				<vertical>
-				<samples>50</samples>
+				<samples>12</samples>
 				<resolution>1</resolution>
 				<min_angle>${-7.22/180*M_PI}</min_angle>
