Commit message: 学习维哥代码，改了一下launch文件，将局部路径规划订阅的点云转为自己写的节点，原来那个不知道是不是滤波了>_<

File: src/sentry_laser_sim/xacro/sentry_sim.xacro (robot description, xacro)
@@ -22,7 +22,7 @@
 <!--base_link->laser_link-->
 <xacro:myjoint_fixed joint_name="laser_joint" joint_type="fixed" x="0" y="0" z="0.135" wx="0" wz="0" wy="0" parent_link="base_link_sentry" child_link="laser_link"/>
-<link name="base_link">
+<!-- <link name="base_link">
    </link>
-<xacro:myjoint_fixed joint_name="gmapping_joint" joint_type="fixed" x="0" y="0" z="0.0" wx="0" wz="0" wy="0" parent_link="base_footprint" child_link="base_link"/>
+<xacro:myjoint_fixed joint_name="gmapping_joint" joint_type="fixed" x="0" y="0" z="0.0" wx="0" wz="0" wy="0" parent_link="base_footprint" child_link="base_link"/> -->
 <!-- 每一个驱动轮都需要配置传动装置 -->
     <xacro:joint_trans joint_name="base_to_wheel_l_f"/>
