Commit message: 添加了小陀螺；点云分割；简易版舵轮仿真;...

File: src/sentry_laser_sim/xacro/fun_define.xacro (robot description, xacro)
@@ -67,5 +67,5 @@
 </xacro:macro>
 <!-- 传动实现:用于连接控制器与关节 -->
-    <xacro:macro name="joint_trans" params="joint_name">
+    <xacro:macro name="joint_trans_v" params="joint_name">
         <!-- Transmission is important to link the joints and the controller -->
         <transmission name="${joint_name}_trans">
@@ -80,3 +80,15 @@
         </transmission>
     </xacro:macro>
+<!-- 传动实现:用于连接控制器与关节 -->
+    <xacro:macro name="joint_trans_e" params="joint_name">
+    <transmission name="trans_${joint_name}">
+      <type>transmission_interface/SimpleTransmission</type>
+      <actuator name="${joint_name}_actuator">
+        <mechanicalReduction>1</mechanicalReduction>
+      </actuator>
+      <joint name="${joint_name}">
+        <hardwareInterface>hardware_interface/EffortJointInterface</hardwareInterface>
+      </joint>
+    </transmission>
+    </xacro:macro>
 </robot>

File: src/sentry_laser_sim/xacro/laser.xacro (robot description, xacro)
@@ -3,7 +3,7 @@
 <xacro:include filename="$(find sentry_laser_sim)/xacro/fun_define.xacro"/>
 <!--laser_link-->
-<xacro:mylink_tri myname="laser_link" l="0.1" w="0.1" h="0.05" x="0" y="0" z="0" wx="0" wy="0" wz="0" color="red" r="0" g="0" b="0" a="1" mass="1" ixx="1.0" ixy="0.0" ixz="0.0" iyy="1.0" iyz="0.0" izz="1.0"/>
+<xacro:mylink_tri myname="laser_link" l="0.1" w="0.1" h="0.05" x="0" y="0" z="0" wx="0" wy="0" wz="0" color="red" r="0" g="0" b="0" a="1" mass="3" ixx="0.01" ixy="0.0" ixz="0.0" iyy="0.01" iyz="0.0" izz="0.01"/>
 <!--laser_fake_link-->
-<xacro:mylink_tri myname="laser_fake_link" l="0.001" w="0.001" h="0.001" x="0" y="0" z="0" wx="0" wy="0" wz="0" color="red" r="0" g="0" b="0" a="1" mass="0.001" ixx="0.0" ixy="0.0" ixz="0.0" iyy="0.0" iyz="0.0" izz="0.0"/>
+<!-- <xacro:mylink_tri myname="laser_fake_link" l="0.001" w="0.001" h="0.001" x="0" y="0" z="0" wx="0" wy="0" wz="0" color="red" r="0" g="0" b="0" a="1" mass="0.001" ixx="0.0" ixy="0.0" ixz="0.0" iyy="0.0" iyz="0.0" izz="0.0"/> -->
 <!--livox_laser_simulation-->
 <xacro:property name="M_PI" value="3.14159"/>
@@ -22,7 +22,7 @@
   </xacro:macro>
   <xacro:macro name="Livox_Mid_gazebo_sensor" params="visualize:=True update_rate:=10 resolution:=0.002 noise_mean:=0.0 noise_stddev:=0.00 name:=laser">
-    <gazebo reference="${name}_fake_link">
+    <gazebo reference="${name}_link">
       <sensor type="ray" name="${name}_livox">
-        <pose>0 0 3 0 0 0</pose>
+        <pose>0 0 0 0 0 0</pose>
         <visualize>${visualize}</visualize>
         <update_rate>10</update_rate>
@@ -64,3 +64,22 @@
   </xacro:macro>
     <xacro:Livox_Mid_gazebo_sensor name="laser" visualize="true"/>
+<gazebo reference="laser_link">
+        <gravity>true</gravity>
+        <sensor name="imu_sensor" type="imu">
+            <always_on>true</always_on>
+            <update_rate>100</update_rate>
+            <visualize>true</visualize>
+            <topic>__default_topic__</topic>
+            <plugin filename="libgazebo_ros_imu_sensor.so" name="imu_plugin">
+                <topicName>imu</topicName>
+                <bodyName>imu</bodyName>
+                <updateRateHZ>100.0</updateRateHZ>
+                <gaussianNoise>0.0</gaussianNoise>
+                <xyzOffset>0 0 0</xyzOffset>
+                <rpyOffset>0 0 0</rpyOffset>
+                <frameName>imu</frameName>
+            </plugin>
+            <pose>0 0 0 0 0 0</pose>
+        </sensor>
+    </gazebo>
 </robot>

File: src/sentry_laser_sim/xacro/sentry_sim.xacro (robot description, xacro)
@@ -2,5 +2,5 @@
 <robot xmlns:xacro="http://www.ros.org/wiki/xacro" name="car_laser">
     <xacro:include filename="$(find sentry_laser_sim)/xacro/base_link.xacro" />
-    <xacro:include filename="$(find sentry_laser_sim)/xacro/imu.xacro" />
+    <!-- <xacro:include filename="$(find sentry_laser_sim)/xacro/imu.xacro" /> -->
     <xacro:include filename="$(find sentry_laser_sim)/xacro/laser.xacro" />
     <xacro:include filename="$(find sentry_laser_sim)/xacro/wheel.xacro" />
@@ -15,19 +15,34 @@
 <xacro:myjoint_continuous joint_name="base_to_wheel_r_b" joint_type="continuous" x="-0.1" y="-0.125" z="0" wx="0" wy="0" wz="0" parent_link="base_link_sentry" child_link="wheel_r_b" ax="0" ay="-1" az="0"/>
 <!--base_footprint->base_link-->
-<xacro:myjoint_fixed joint_name="base_footprint_joint" joint_type="fixed" x="0" y="0" z="0.1" wx="0" wz="0" wy="0" parent_link="base_footprint" child_link="base_link_sentry"/>
+<xacro:myjoint_fixed joint_name="base_footprint_joint" joint_type="fixed" x="0" y="0" z="0.1" wx="0" wz="0.0" wy="0" parent_link="base_footprint" child_link="base_link_sentry"/>
 <!--base_footprint->laser_fake_link-->
-<xacro:myjoint_fixed joint_name="fake_laser_joint" joint_type="fixed" x="0" y="0" z="0.135" wx="0" wz="0" wy="0" parent_link="base_link_sentry" child_link="laser_fake_link"/>
+<!-- <xacro:myjoint_fixed joint_name="fake_laser_joint" joint_type="fixed" x="0" y="0" z="0.135" wx="0" wz="0" wy="0" parent_link="base_link_sentry" child_link="laser_fake_link"/> -->
 <!--base_link->camera_link-->
-<xacro:myjoint_fixed joint_name="imu_joint" joint_type="fixed" x="0.175" y="0" z="0" wx="0" wz="0" wy="0" parent_link="base_link_sentry" child_link="imu_link"/>
+<!-- <xacro:myjoint_fixed joint_name="imu_joint" joint_type="fixed" x="0.0" y="0" z="0" wx="0" wz="0" wy="0" parent_link="base_link_sentry" child_link="imu_link"/> -->
 <!--base_link->laser_link-->
-<xacro:myjoint_fixed joint_name="laser_joint" joint_type="fixed" x="0" y="0" z="0.135" wx="0" wz="0" wy="0" parent_link="base_link_sentry" child_link="laser_link"/>
+<!-- <xacro:myjoint_fixed joint_name="laser_joint" joint_type="fixed" x="0" y="0" z="0.135" wx="0" wz="0" wy="0" parent_link="base_link_sentry" child_link="laser_link"/> -->
+<xacro:myjoint_continuous joint_name="yaw_joint" joint_type="continuous" x="0.05" y="0.0" z="0.135" wx="0" wy="0" wz="0" parent_link="base_link_sentry" child_link="laser_link" ax="0" ay="0" az="1"/>
 <!-- <link name="base_link">
    </link>
 <xacro:myjoint_fixed joint_name="gmapping_joint" joint_type="fixed" x="0" y="0" z="0.0" wx="0" wz="0" wy="0" parent_link="base_footprint" child_link="base_link"/> -->
 <!-- 每一个驱动轮都需要配置传动装置 -->
-    <xacro:joint_trans joint_name="base_to_wheel_l_f"/>
-    <xacro:joint_trans joint_name="base_to_wheel_l_b" />
-    <xacro:joint_trans joint_name="base_to_wheel_r_f" />
-    <xacro:joint_trans joint_name="base_to_wheel_r_b" />
+    <xacro:joint_trans_v joint_name="base_to_wheel_l_f"/>
+    <xacro:joint_trans_v joint_name="base_to_wheel_l_b" />
+    <xacro:joint_trans_v joint_name="base_to_wheel_r_f" />
+    <xacro:joint_trans_v joint_name="base_to_wheel_r_b" />
+    <xacro:joint_trans_e joint_name="yaw_joint" />
+  <gazebo>
+    <plugin name="gazebo_ros_control" filename="libgazebo_ros_control.so">
+                <rosDebugLevel>Debug</rosDebugLevel>
+                <publishWheelTF>true</publishWheelTF>
+                <robotNamespace>/sentry</robotNamespace>
+                <robotSimType>gazebo_ros_control/DefaultRobotHWSim</robotSimType>
+                <publishTf>1</publishTf>
+                <publishWheelJointState>true</publishWheelJointState>
+                <alwaysOn>true</alwaysOn>
+                <updateRate>100.0</updateRate>
+                <legacyMode>true</legacyMode>
+    </plugin>
+  </gazebo>
 <gazebo>
 	<plugin name="mecanum_controller" filename="libgazebo_ros_planar_move.so">
@@ -35,9 +50,10 @@
             <odometryTopic>odom</odometryTopic>
            	<odometryFrame>odom</odometryFrame>
+            <robotNamespace>/sentry</robotNamespace>
            	<leftFrontJoint>base_to_wheel_l_f</leftFrontJoint>
            	<rightFrontJoint>base_to_wheel_r_f</rightFrontJoint>
            	<leftRearJoint>base_to_wheel_l_b</leftRearJoint>
-		<rightRearJoint>base_to_wheel_r_b</rightRearJoint>
-		<odometryRate>30</odometryRate>
+		    <rightRearJoint>base_to_wheel_r_b</rightRearJoint>
+		    <odometryRate>30</odometryRate>
            	<robotBaseFrame>base_footprint</robotBaseFrame>
            	<broadcastTF>1</broadcastTF>

File: src/sentry_laser_sim/xacro_simple_sentry/simple_sentry.xacro (robot description, xacro)
@@ -97,8 +97,6 @@
                 <publishWheelJointState>true</publishWheelJointState>
                 <alwaysOn>true</alwaysOn>
-                <updateRate>100.0</updateRate>
+                <updateRate>20.0</updateRate>
                 <legacyMode>true</legacyMode>
-                <odometryFrame>odom</odometryFrame>
-                <odometryTopic>odom</odometryTopic>
     </plugin>
   </gazebo>
