Commit message: 跑通维哥代码

File: src/sentry_laser_sim/xacro/base_link.xacro (robot description, xacro)
@@ -3,6 +3,6 @@
 <xacro:include filename="$(find sentry_laser_sim)/xacro/fun_define.xacro"/>
 <!--base_link-->
-<xacro:mylink_tri myname="base_link" l="0.3" w="0.2" h="0.1" x="0" y="0" z="0.04" wx="0" wy="0" wz="0" color="red" r="255" g="0" b="0" a="1" mass="100" ixx="1.0" ixy="0.0" ixz="0.0" iyy="1.0" iyz="0.0" izz="1.0"/>
-<gazebo reference="base_link">
+<xacro:mylink_tri myname="base_link_sentry" l="0.3" w="0.2" h="0.1" x="0" y="0" z="0.04" wx="0" wy="0" wz="0" color="red" r="255" g="0" b="0" a="1" mass="100" ixx="1.0" ixy="0.0" ixz="0.0" iyy="1.0" iyz="0.0" izz="1.0"/>
+<gazebo reference="base_link_sentry">
         <material>Gazebo/Green</material>
 </gazebo>

File: src/sentry_laser_sim/xacro/laser.xacro (robot description, xacro)
@@ -8,8 +8,8 @@
 <!--livox_laser_simulation-->
 <xacro:property name="M_PI" value="3.14159"/>
-  <xacro:property name="laser_min_range" value="0.1"/>
-  <xacro:property name="laser_max_range" value="200.0"/>
+  <xacro:property name="laser_min_range" value="0.4"/>
+  <xacro:property name="laser_max_range" value="30.0"/>
   <xacro:property name="ros_topic" value="scan1"/>
-  <xacro:property name="samples" value="10000"/>
+  <xacro:property name="samples" value="24000"/>
   <xacro:property name="downsample" value="0"/>
   <xacro:macro name="null_inertial">
@@ -21,5 +21,5 @@
     </inertial>
   </xacro:macro>
-  <xacro:macro name="Livox_Mid_gazebo_sensor" params="visualize:=True update_rate:=10 resolution:=0.002 noise_mean:=0.0 noise_stddev:=0.01 name:=laser">
+  <xacro:macro name="Livox_Mid_gazebo_sensor" params="visualize:=True update_rate:=10 resolution:=0.002 noise_mean:=0.0 noise_stddev:=0.00 name:=laser">
     <gazebo reference="${name}_fake_link">
       <sensor type="ray" name="${name}_livox">

File: src/sentry_laser_sim/xacro/sentry_sim.xacro (robot description, xacro)
@@ -7,19 +7,19 @@
     <xacro:include filename="$(find sentry_laser_sim)/xacro/fun_define.xacro" />
 <!--base_link->wheel_l_f-->
-<xacro:myjoint_continuous joint_name="base_to_wheel_l_f" joint_type="continuous" x="0.1" y="0.125" z="0" wx="0" wy="0" wz="0" parent_link="base_link" child_link="wheel_l_f" ax="0" ay="1" az="0"/>
+<xacro:myjoint_continuous joint_name="base_to_wheel_l_f" joint_type="continuous" x="0.1" y="0.125" z="0" wx="0" wy="0" wz="0" parent_link="base_link_sentry" child_link="wheel_l_f" ax="0" ay="1" az="0"/>
 <!--base_link->wheel_r_f-->
-<xacro:myjoint_continuous joint_name="base_to_wheel_r_f" joint_type="continuous" x="0.1" y="-0.125" z="0" wx="0" wy="0" wz="0" parent_link="base_link" child_link="wheel_r_f" ax="0" ay="-1" az="0"/>
+<xacro:myjoint_continuous joint_name="base_to_wheel_r_f" joint_type="continuous" x="0.1" y="-0.125" z="0" wx="0" wy="0" wz="0" parent_link="base_link_sentry" child_link="wheel_r_f" ax="0" ay="-1" az="0"/>
 <!--base_link->wheel_l_b-->
-<xacro:myjoint_continuous joint_name="base_to_wheel_l_b" joint_type="continuous" x="-0.1" y="0.125" z="0" wx="0" wy="0" wz="0" parent_link="base_link" child_link="wheel_l_b" ax="0" ay="1" az="0"/>
+<xacro:myjoint_continuous joint_name="base_to_wheel_l_b" joint_type="continuous" x="-0.1" y="0.125" z="0" wx="0" wy="0" wz="0" parent_link="base_link_sentry" child_link="wheel_l_b" ax="0" ay="1" az="0"/>
 <!--base_link->wheel_r_b-->
-<xacro:myjoint_continuous joint_name="base_to_wheel_r_b" joint_type="continuous" x="-0.1" y="-0.125" z="0" wx="0" wy="0" wz="0" parent_link="base_link" child_link="wheel_r_b" ax="0" ay="-1" az="0"/>
+<xacro:myjoint_continuous joint_name="base_to_wheel_r_b" joint_type="continuous" x="-0.1" y="-0.125" z="0" wx="0" wy="0" wz="0" parent_link="base_link_sentry" child_link="wheel_r_b" ax="0" ay="-1" az="0"/>
 <!--base_footprint->base_link-->
-<xacro:myjoint_fixed joint_name="base_footprint_joint" joint_type="fixed" x="0" y="0" z="0.5" wx="0" wz="0" wy="0" parent_link="base_footprint" child_link="base_link"/>
+<xacro:myjoint_fixed joint_name="base_footprint_joint" joint_type="fixed" x="0" y="0" z="0.1" wx="0" wz="0" wy="0" parent_link="base_footprint" child_link="base_link_sentry"/>
 <!--base_footprint->laser_fake_link-->
-<xacro:myjoint_fixed joint_name="fake_laser_joint" joint_type="fixed" x="0" y="0" z="0.135" wx="0" wz="0" wy="0" parent_link="base_link" child_link="laser_fake_link"/>
+<xacro:myjoint_fixed joint_name="fake_laser_joint" joint_type="fixed" x="0" y="0" z="0.135" wx="0" wz="0" wy="0" parent_link="base_link_sentry" child_link="laser_fake_link"/>
 <!--base_link->camera_link-->
-<xacro:myjoint_fixed joint_name="imu_joint" joint_type="fixed" x="0.175" y="0" z="0" wx="0" wz="0" wy="0" parent_link="base_link" child_link="imu_link"/>
+<xacro:myjoint_fixed joint_name="imu_joint" joint_type="fixed" x="0.175" y="0" z="0" wx="0" wz="0" wy="0" parent_link="base_link_sentry" child_link="imu_link"/>
 <!--base_link->laser_link-->
-<xacro:myjoint_fixed joint_name="laser_joint" joint_type="fixed" x="0" y="0" z="0.135" wx="0" wz="0" wy="0" parent_link="base_link" child_link="laser_link"/>
+<xacro:myjoint_fixed joint_name="laser_joint" joint_type="fixed" x="0" y="0" z="0.135" wx="0" wz="0" wy="0" parent_link="base_link_sentry" child_link="laser_link"/>
 <!--camera_link->fake_link_kinect-->
 <!--Camera_Control-->
@@ -76,6 +76,6 @@
 	<plugin name="mecanum_controller" filename="libgazebo_ros_planar_move.so">
 		<commandTopic>cmd_vel</commandTopic>
-                <odometryTopic>odom</odometryTopic>
-           	<odometryFrame>odom</odometryFrame>
+            <odometryTopic>odom_sentry</odometryTopic>
+           	<odometryFrame>odom_sentry</odometryFrame>
            	<leftFrontJoint>base_to_wheel_l_f</leftFrontJoint>
            	<rightFrontJoint>base_to_wheel_r_f</rightFrontJoint>

Commit message: 更新

File: src/sentry_laser_sim/xacro/base_link.xacro (robot description, xacro)
@@ -3,5 +3,5 @@
 <xacro:include filename="$(find sentry_laser_sim)/xacro/fun_define.xacro"/>
 <!--base_link-->
-<xacro:mylink_tri myname="base_link_sentry" l="0.3" w="0.2" h="0.1" x="0" y="0" z="0.04" wx="0" wy="0" wz="0" color="red" r="255" g="0" b="0" a="1" mass="100" ixx="1.0" ixy="0.0" ixz="0.0" iyy="1.0" iyz="0.0" izz="1.0"/>
+<xacro:mylink_tri myname="base_link_sentry" l="0.3" w="0.2" h="0.1" x="0" y="0" z="0.04" wx="0" wy="0" wz="0" color="red" r="255" g="0" b="0" a="1" mass="50" ixx="1" ixy="0.0" ixz="0.0" iyy="1" iyz="0.0" izz="1"/>
 <gazebo reference="base_link_sentry">
         <material>Gazebo/Green</material>

File: src/sentry_laser_sim/xacro/imu.xacro (robot description, xacro)
@@ -2,5 +2,5 @@
 <robot xmlns:xacro="http://www.ros.org/wiki/xacro" name="imu">
 <!--camera_link-->
-<xacro:mylink_tri myname="imu_link" l="0.05" w="0.15" h="0.05" x="0" y="0" z="0.04" wx="0" wy="0" wz="0" color="red" r="0" g="0" b="0" a="1" mass="1" ixx="1.0" ixy="0.0" ixz="0.0" iyy="1.0" iyz="0.0" izz="1.0"/>
+<xacro:mylink_tri myname="imu_link" l="0.05" w="0.15" h="0.05" x="0" y="0" z="0.04" wx="0" wy="0" wz="0" color="red" r="0" g="0" b="0" a="1" mass="0.1" ixx="0.001" ixy="0.0" ixz="0.0" iyy="0.001" iyz="0.0" izz="0.001"/>
 <gazebo reference="imu_link">
         <gravity>true</gravity>

File: src/sentry_laser_sim/xacro/laser.xacro (robot description, xacro)
@@ -3,5 +3,5 @@
 <xacro:include filename="$(find sentry_laser_sim)/xacro/fun_define.xacro"/>
 <!--laser_link-->
-<xacro:mylink_tri myname="laser_link" l="0.1" w="0.1" h="0.05" x="0" y="0" z="0" wx="0" wy="0" wz="0" color="red" r="0" g="0" b="0" a="1" mass="3" ixx="0.01" ixy="0.0" ixz="0.0" iyy="0.01" iyz="0.0" izz="0.01"/>
+<xacro:mylink_tri myname="laser_link" l="0.1" w="0.1" h="0.05" x="0" y="0" z="0" wx="0" wy="0" wz="0" color="red" r="0" g="0" b="0" a="1" mass="0.1" ixx="0.001" ixy="0.0" ixz="0.0" iyy="0.001" iyz="0.0" izz="0.001"/>
 <!--laser_fake_link-->
 <!-- <xacro:mylink_tri myname="laser_fake_link" l="0.001" w="0.001" h="0.001" x="0" y="0" z="0" wx="0" wy="0" wz="0" color="red" r="0" g="0" b="0" a="1" mass="0.001" ixx="0.0" ixy="0.0" ixz="0.0" iyy="0.0" iyz="0.0" izz="0.0"/> -->
@@ -11,5 +11,5 @@
   <xacro:property name="laser_max_range" value="30.0"/>
   <xacro:property name="ros_topic" value="scan1"/>
-  <xacro:property name="samples" value="24000"/>
+  <xacro:property name="samples" value="60000"/>
   <xacro:property name="downsample" value="0"/>
   <xacro:macro name="null_inertial">

File: src/sentry_laser_sim/xacro/sentry_sim.xacro (robot description, xacro)
@@ -56,5 +56,5 @@
 		    <rightRearJoint>base_to_wheel_r_b</rightRearJoint>
 		    <odometryRate>30</odometryRate>
-           	<robotBaseFrame>base_footprint</robotBaseFrame>
+           	<robotBaseFrame>base_link_sentry</robotBaseFrame>
            	<broadcastTF>1</broadcastTF>
         </plugin>

File: src/sentry_laser_sim/xacro/wheel.xacro (robot description, xacro)
@@ -3,20 +3,20 @@
 <xacro:include filename="$(find sentry_laser_sim)/xacro/fun_define.xacro"/>
 <!--wheel_l_f-->
-<xacro:mylink_cyl link_name="wheel_l_f" l="0.05" r_="0.05" x="0" y="0" z="0" wx="${M_PI/2}" wy="0" wz="0" color="bule" r="0" g="0" b="255" a="1" mass="10" ixx="1.0" ixy="0.0" ixz="0.0" iyy="1.0" iyz="0.0" izz="1.0"/>
+<xacro:mylink_cyl link_name="wheel_l_f" l="0.05" r_="0.05" x="0" y="0" z="0" wx="${M_PI/2}" wy="0" wz="0" color="bule" r="0" g="0" b="255" a="1" mass="0.1" ixx="0.001" ixy="0.0" ixz="0.0" iyy="0.001" iyz="0.0" izz="0.001"/>
 <gazebo reference="wheel_l_f">
         <material>Gazebo/Red</material>
 </gazebo>
 <!--wheel_r_f-->
-<xacro:mylink_cyl link_name="wheel_r_f" l="0.05" r_="0.05" x="0" y="0" z="0" wx="${M_PI/2}" wy="0" wz="0" color="bule" r="255" g="0" b="255" a="1" mass="10" ixx="1.0" ixy="0.0" ixz="0.0" iyy="1.0" iyz="0.0" izz="1.0"/>
+<xacro:mylink_cyl link_name="wheel_r_f" l="0.05" r_="0.05" x="0" y="0" z="0" wx="${M_PI/2}" wy="0" wz="0" color="bule" r="255" g="0" b="255" a="1" mass="0.1" ixx="0.001" ixy="0.0" ixz="0.0" iyy="0.001" iyz="0.0" izz="0.001"/>
 <gazebo reference="wheel_r_f">
         <material>Gazebo/Red</material>
 </gazebo>
 <!--wheel_l_b-->
-<xacro:mylink_cyl link_name="wheel_l_b" l="0.05" r_="0.05" x="0" y="0" z="0" wx="${M_PI/2}" wy="0" wz="0" color="bule" r="0" g="0" b="255" a="1" mass="10" ixx="1.0" ixy="0.0" ixz="0.0" iyy="1.0" iyz="0.0" izz="1.0"/>
+<xacro:mylink_cyl link_name="wheel_l_b" l="0.05" r_="0.05" x="0" y="0" z="0" wx="${M_PI/2}" wy="0" wz="0" color="bule" r="0" g="0" b="255" a="1" mass="0.1" ixx="0.001" ixy="0.0" ixz="0.0" iyy="0.001" iyz="0.0" izz="0.001"/>
 <gazebo reference="wheel_l_b">
         <material>Gazebo/Red</material>
 </gazebo>
 <!--wheel_r_b-->
-<xacro:mylink_cyl link_name="wheel_r_b" l="0.05" r_="0.05" x="0" y="0" z="0" wx="${M_PI/2}" wy="0" wz="0" color="bule" r="0" g="0" b="0" a="1" mass="10" ixx="1.0" ixy="0.0" ixz="0.0" iyy="1.0" iyz="0.0" izz="1.0"/>
+<xacro:mylink_cyl link_name="wheel_r_b" l="0.05" r_="0.05" x="0" y="0" z="0" wx="${M_PI/2}" wy="0" wz="0" color="bule" r="0" g="0" b="0" a="1" mass="0.1" ixx="0.001" ixy="0.0" ixz="0.0" iyy="0.001" iyz="0.0" izz="0.001"/>
 <gazebo reference="wheel_r_b">
         <material>Gazebo/Red</material>
