Commit message: 小改，完善readme

File: src/sentry_kinematics_sim/xacro/livox_sim.xacro (robot description, xacro)
@@ -1,5 +1,5 @@
 <?xml version="1.0"?>
 <robot xmlns:xacro="http://ros.org/wiki/xacro">
-    <xacro:include filename="$(find sentry9)/xacro/sentry_laser.xacro" />
+    <xacro:include filename="$(find sentry_kinematics_sim)/xacro/sentry_laser.xacro" />
   <xacro:property name="M_PI" value="3.14159"/>
   <xacro:property name="laser_min_range" value="0.1"/>
@@ -52,5 +52,5 @@
 		  <samples>${samples}</samples>
 		  <downsample>${downsample}</downsample>
-		  <csv_file_name>package://sentry9/scan_mode/mid360.csv</csv_file_name>
+		  <csv_file_name>package://sentry_laser_sim/scan_mode/mid360.csv</csv_file_name>
 		  <ros_topic>${ros_topic}</ros_topic>
         </plugin>

File: src/sentry_kinematics_sim/xacro/sentry.xacro (robot description, xacro)
@@ -1,13 +1,13 @@
 <?xml version="1.0" encoding="utf-8"?>
 <robot name="sentry" xmlns:xacro="http://www.ros.org/wiki/xacro">
-    <xacro:include filename="$(find sentry9)/xacro/sentry_chassis_new.xacro" />
-    <xacro:include filename="$(find sentry9)/xacro/sentry_yaw.xacro" />
+    <xacro:include filename="$(find sentry_kinematics_sim)/xacro/sentry_chassis_new.xacro" />
+    <xacro:include filename="$(find sentry_kinematics_sim)/xacro/sentry_yaw.xacro" />
     <!--xacro:include filename="$(find sentry9)/xacro/sentry_laser.xacro" /-->
-    <xacro:include filename="$(find sentry9)/xacro/sentry_pitch.xacro" />
-    <xacro:include filename="$(find sentry9)/xacro/sentry_camera.xacro" />
-    <xacro:include filename="$(find sentry9)/xacro/sentry_imu.xacro" />
-    <xacro:include filename="$(find sentry9)/xacro/sentry_trigger.xacro" />
-    <xacro:include filename="$(find sentry9)/xacro/livox_sim.xacro"/>
-    <xacro:include filename="$(find sentry9)/xacro/sentry_wheel.xacro" />
+    <xacro:include filename="$(find sentry_kinematics_sim)/xacro/sentry_pitch.xacro" />
+    <xacro:include filename="$(find sentry_kinematics_sim)/xacro/sentry_camera.xacro" />
+    <xacro:include filename="$(find sentry_kinematics_sim)/xacro/sentry_imu.xacro" />
+    <xacro:include filename="$(find sentry_kinematics_sim)/xacro/sentry_trigger.xacro" />
+    <xacro:include filename="$(find sentry_kinematics_sim)/xacro/livox_sim.xacro"/>
+    <xacro:include filename="$(find sentry_kinematics_sim)/xacro/sentry_wheel.xacro" />
     <!-- Yaw_Joint -->
   <joint

File: src/sentry_kinematics_sim/xacro/sentry_camera.xacro (robot description, xacro)
@@ -23,5 +23,5 @@
       <geometry>
         <mesh
-          filename="package://sentry9/meshes/Camera_Link.STL" />
+          filename="package://sentry_kinematics_sim/meshes/Camera_Link.STL" />
       </geometry>
       <material
@@ -37,5 +37,5 @@
       <geometry>
         <mesh
-          filename="package://sentry9/meshes/Camera_Link.STL" />
+          filename="package://sentry_kinematics_sim/meshes/Camera_Link.STL" />
       </geometry>
     </collision>

File: src/sentry_kinematics_sim/xacro/sentry_chassis.xacro (robot description, xacro)
@@ -23,5 +23,5 @@
       <geometry>
         <mesh
-          filename="package://sentry9/meshes/base_link.STL" />
+          filename="package://sentry_kinematics_sim/meshes/base_link.STL" />
       </geometry>
       <material
@@ -37,5 +37,5 @@
       <geometry>
         <mesh
-          filename="package://sentry9/meshes/base_link.STL" />
+          filename="package://sentry_kinematics_sim/meshes/base_link.STL" />
       </geometry>
     </collision>
@@ -76,5 +76,5 @@
       <geometry>
         <mesh
-          filename="package://sentry9/meshes/Heading_Left_Front_Link.STL" />
+          filename="package://sentry_kinematics_sim/meshes/Heading_Left_Front_Link.STL" />
       </geometry>
       <material
@@ -90,5 +90,5 @@
       <geometry>
         <mesh
-          filename="package://sentry9/meshes/Heading_Left_Front_Link.STL" />
+          filename="package://sentry_kinematics_sim/meshes/Heading_Left_Front_Link.STL" />
       </geometry>
     </collision>
@@ -129,5 +129,5 @@
       <geometry>
         <mesh
-          filename="package://sentry9/meshes/Driving_Left_Front_Link.STL" />
+          filename="package://sentry_kinematics_sim/meshes/Driving_Left_Front_Link.STL" />
       </geometry>
       <material
@@ -143,5 +143,5 @@
       <geometry>
         <mesh
-          filename="package://sentry9/meshes/Driving_Left_Front_Link.STL" />
+          filename="package://sentry_kinematics_sim/meshes/Driving_Left_Front_Link.STL" />
       </geometry>
     </collision>
@@ -183,5 +183,5 @@
       <geometry>
         <mesh
-          filename="package://sentry9/meshes/Heading_Left_Back_link.STL" />
+          filename="package://sentry_kinematics_sim/meshes/Heading_Left_Back_link.STL" />
       </geometry>
       <material
@@ -197,5 +197,5 @@
       <geometry>
         <mesh
-          filename="package://sentry9/meshes/Heading_Left_Back_link.STL" />
+          filename="package://sentry_kinematics_sim/meshes/Heading_Left_Back_link.STL" />
       </geometry>
     </collision>
@@ -236,5 +236,5 @@
       <geometry>
         <mesh
-          filename="package://sentry9/meshes/Driving_Left_back_Link.STL" />
+          filename="package://sentry_kinematics_sim/meshes/Driving_Left_back_Link.STL" />
       </geometry>
       <material
@@ -250,5 +250,5 @@
       <geometry>
         <mesh
-          filename="package://sentry9/meshes/Driving_Left_back_Link.STL" />
+          filename="package://sentry_kinematics_sim/meshes/Driving_Left_back_Link.STL" />
       </geometry>
     </collision>
@@ -290,5 +290,5 @@
       <geometry>
         <mesh
-          filename="package://sentry9/meshes/Heading_Right_Front_link.STL" />
+          filename="package://sentry_kinematics_sim/meshes/Heading_Right_Front_link.STL" />
       </geometry>
       <material
@@ -304,5 +304,5 @@
       <geometry>
         <mesh
-          filename="package://sentry9/meshes/Heading_Right_Front_link.STL" />
+          filename="package://sentry_kinematics_sim/meshes/Heading_Right_Front_link.STL" />
       </geometry>
     </collision>
@@ -343,5 +343,5 @@
       <geometry>
         <mesh
-          filename="package://sentry9/meshes/Driving_Right_Front_Link.STL" />
+          filename="package://sentry_kinematics_sim/meshes/Driving_Right_Front_Link.STL" />
       </geometry>
       <material
@@ -357,5 +357,5 @@
       <geometry>
         <mesh
-          filename="package://sentry9/meshes/Driving_Right_Front_Link.STL" />
+          filename="package://sentry_kinematics_sim/meshes/Driving_Right_Front_Link.STL" />
       </geometry>
     </collision>
@@ -397,5 +397,5 @@
       <geometry>
         <mesh
-          filename="package://sentry9/meshes/Heading_Right_Back_Link.STL" />
+          filename="package://sentry_kinematics_sim/meshes/Heading_Right_Back_Link.STL" />
       </geometry>
       <material
@@ -411,5 +411,5 @@
       <geometry>
         <mesh
-          filename="package://sentry9/meshes/Heading_Right_Back_Link.STL" />
+          filename="package://sentry_kinematics_sim/meshes/Heading_Right_Back_Link.STL" />
       </geometry>
     </collision>
@@ -450,5 +450,5 @@
       <geometry>
         <mesh
-          filename="package://sentry9/meshes/Driving_Right_Back_Link.STL" />
+          filename="package://sentry_kinematics_sim/meshes/Driving_Right_Back_Link.STL" />
       </geometry>
       <material
@@ -464,5 +464,5 @@
       <geometry>
         <mesh
-          filename="package://sentry9/meshes/Driving_Right_Back_Link.STL" />
+          filename="package://sentry_kinematics_sim/meshes/Driving_Right_Back_Link.STL" />
       </geometry>
     </collision>

File: src/sentry_kinematics_sim/xacro/sentry_chassis_new.xacro (robot description, xacro)
@@ -23,5 +23,5 @@
       <geometry>
         <mesh
-          filename="package://sentry9/meshes/base_link.STL" />
+          filename="package://sentry_kinematics_sim/meshes/base_link.STL" />
       </geometry>
       <material
@@ -37,5 +37,5 @@
       <geometry>
         <mesh
-          filename="package://sentry9/meshes/base_link.STL" />
+          filename="package://sentry_kinematics_sim/meshes/base_link.STL" />
       </geometry>
     </collision>

File: src/sentry_kinematics_sim/xacro/sentry_imu.xacro (robot description, xacro)
@@ -23,5 +23,5 @@
       <geometry>
         <mesh
-          filename="package://sentry9/meshes/IMU_Link.STL" />
+          filename="package://sentry_kinematics_sim/meshes/IMU_Link.STL" />
       </geometry>
       <material
@@ -37,5 +37,5 @@
       <geometry>
         <mesh
-          filename="package://sentry9/meshes/IMU_Link.STL" />
+          filename="package://sentry_kinematics_sim/meshes/IMU_Link.STL" />
       </geometry>
     </collision>

File: src/sentry_kinematics_sim/xacro/sentry_laser.xacro (robot description, xacro)
@@ -23,5 +23,5 @@
       <geometry>
         <mesh
-          filename="package://sentry9/meshes/Laser_Link.STL" />
+          filename="package://sentry_kinematics_sim/meshes/Laser_Link.STL" />
       </geometry>
       <material
@@ -37,5 +37,5 @@
       <geometry>
         <mesh
-          filename="package://sentry9/meshes/Laser_Link.STL" />
+          filename="package://sentry_kinematics_sim/meshes/Laser_Link.STL" />
       </geometry>
     </collision>

File: src/sentry_kinematics_sim/xacro/sentry_pitch.xacro (robot description, xacro)
@@ -23,5 +23,5 @@
       <geometry>
         <mesh
-          filename="package://sentry9/meshes/Pitch_Link.STL" />
+          filename="package://sentry_kinematics_sim/meshes/Pitch_Link.STL" />
       </geometry>
       <material
@@ -37,5 +37,5 @@
       <geometry>
         <mesh
-          filename="package://sentry9/meshes/Pitch_Link.STL" />
+          filename="package://sentry_kinematics_sim/meshes/Pitch_Link.STL" />
       </geometry>
     </collision>

File: src/sentry_kinematics_sim/xacro/sentry_trigger.xacro (robot description, xacro)
@@ -23,5 +23,5 @@
       <geometry>
         <mesh
-          filename="package://sentry9/meshes/Left_Trigger_Link.STL" />
+          filename="package://sentry_kinematics_sim/meshes/Left_Trigger_Link.STL" />
       </geometry>
       <material
@@ -37,5 +37,5 @@
       <geometry>
         <mesh
-          filename="package://sentry9/meshes/Left_Trigger_Link.STL" />
+          filename="package://sentry_kinematics_sim/meshes/Left_Trigger_Link.STL" />
       </geometry>
     </collision>
@@ -63,5 +63,5 @@
       <geometry>
         <mesh
-          filename="package://sentry9/meshes/Rigth_Trigger_Link.STL" />
+          filename="package://sentry_kinematics_sim/meshes/Rigth_Trigger_Link.STL" />
       </geometry>
       <material
@@ -77,5 +77,5 @@
       <geometry>
         <mesh
-          filename="package://sentry9/meshes/Rigth_Trigger_Link.STL" />
+          filename="package://sentry_kinematics_sim/meshes/Rigth_Trigger_Link.STL" />
       </geometry>
     </collision>

File: src/sentry_kinematics_sim/xacro/sentry_wheel.xacro (robot description, xacro)
@@ -35,5 +35,5 @@
       <geometry>
         <mesh
-          filename="package://sentry9/meshes/Heading_Left_Front_Link.STL" />
+          filename="package://sentry_kinematics_sim/meshes/Heading_Left_Front_Link.STL" />
       </geometry>
       <material
@@ -49,5 +49,5 @@
       <geometry>
         <mesh
-          filename="package://sentry9/meshes/Heading_Left_Front_Link.STL" />
+          filename="package://sentry_kinematics_sim/meshes/Heading_Left_Front_Link.STL" />
       </geometry>
     </collision>
@@ -88,5 +88,5 @@
       <geometry>
         <mesh
-          filename="package://sentry9/meshes/Driving_Left_Front_Link.STL" />
+          filename="package://sentry_kinematics_sim/meshes/Driving_Left_Front_Link.STL" />
       </geometry>
       <material
@@ -102,5 +102,5 @@
       <geometry>
         <mesh
-          filename="package://sentry9/meshes/Driving_Left_Front_Link.STL" />
+          filename="package://sentry_kinematics_sim/meshes/Driving_Left_Front_Link.STL" />
       </geometry>
     </collision>

File: src/sentry_kinematics_sim/xacro/sentry_yaw.xacro (robot description, xacro)
@@ -23,5 +23,5 @@
       <geometry>
         <mesh
-          filename="package://sentry9/meshes/Yaw_Link.STL" />
+          filename="package://sentry_kinematics_sim/meshes/Yaw_Link.STL" />
       </geometry>
       <material
@@ -37,5 +37,5 @@
       <geometry>
         <mesh
-          filename="package://sentry9/meshes/Yaw_Link.STL" />
+          filename="package://sentry_kinematics_sim/meshes/Yaw_Link.STL" />
       </geometry>
     </collision>

File: src/sentry_laser_sim/xacro/sentry_sim.xacro (robot description, xacro)
@@ -22,50 +22,7 @@
 <!--base_link->laser_link-->
 <xacro:myjoint_fixed joint_name="laser_joint" joint_type="fixed" x="0" y="0" z="0.135" wx="0" wz="0" wy="0" parent_link="base_link_sentry" child_link="laser_link"/>
-<!--camera_link->fake_link_kinect-->
-<!--Camera_Control-->
-  <!--gazebo reference="camera_link">
-    <material>Gazebo/Black</material>
-  </gazebo>
-  <gazebo reference="camera_link">
-    <sensor type="depth" name="camera_link">
-      <always_on>true</always_on>
-      <update_rate>30.0</update_rate>
-      <camera name="head">
-	<horizontal_fov>1.3962634</horizontal_fov>
-	<image>
-	  <width>1280</width>
-	  <height>720</height>
-	  <format>R8G8B8</format>
-	</image>
-	<clip>
-	  <near>0.02</near>
-	  <far>300</far>
-	</clip>
-	<noise>
-	  <type>gaussian</type>
-	  <mean>0.0</mean>
-	  <stddev>0.007</stddev>
-	</noise>
-      </camera>
-          <plugin name="kinect_Camera_controller" filename="libgazebo_ros_openni_kinect.so">
-              <cameraName>Kinect_camera</cameraName>
-              <alwaysOn>true</alwaysOn>
-              <updateRate>10</updateRate>
-              <imageTopicName>rgb/image_raw</imageTopicName>
-              <depthImageTopicName>depth/image_raw</depthImageTopicName>
-              <pointCloudTopicName>depth/points</pointCloudTopicName>
-              <cameraInfoTopicName>rgb/camera_info</cameraInfoTopicName>
-              <depthImageCameraInfoTopicName>depth/camera_info</depthImageCameraInfoTopicName>
-              <frameName>fake_link_kinect</frameName>
-              <baseline>0.1</baseline>
-              <distortion_k1>0.0</distortion_k1>
-              <distortion_k2>0.0</distortion_k2>
-              <distortion_k3>0.0</distortion_k3>
-              <distortion_t1>0.0</distortion_t1>
-              <distortion_t2>0.0</distortion_t2>
-              <pointCloudCutoff>0.4</pointCloudCutoff>
-          </plugin>
-    </sensor>
-  </gazebo-->
+<link name="base_link">
+   </link>
+<xacro:myjoint_fixed joint_name="gmapping_joint" joint_type="fixed" x="0" y="0" z="0.0" wx="0" wz="0" wy="0" parent_link="base_footprint" child_link="base_link"/>
 <!-- 每一个驱动轮都需要配置传动装置 -->
     <xacro:joint_trans joint_name="base_to_wheel_l_f"/>
@@ -76,6 +33,6 @@
 	<plugin name="mecanum_controller" filename="libgazebo_ros_planar_move.so">
 		<commandTopic>cmd_vel</commandTopic>
-            <odometryTopic>odom_sentry</odometryTopic>
-           	<odometryFrame>odom_sentry</odometryFrame>
+            <odometryTopic>odom</odometryTopic>
+           	<odometryFrame>odom</odometryFrame>
            	<leftFrontJoint>base_to_wheel_l_f</leftFrontJoint>
            	<rightFrontJoint>base_to_wheel_r_f</rightFrontJoint>
